File: kwp1281_tool/hardware/kicad/kwp1281tool/kwp1281tool.kicad_sch (KiCad schematic)
At the start: 23 parts, among them J1 AVR-JTAG-10, J2 TTL-232R-5V, J3 Conn_01x04_Male, SW1 SW_Omron_B3FS, U1 L9637D, U2 LD1117S50CTR, U3 ATmega1284-P, U4 ISO6721BQDRQ1, Y1 18.432 MHz

Commit message: Integrate USB onto the board
Parts:
- removed J2: TTL-232R-5V, Connector_PinHeader_2.54mm:PinHeader_1x06_P2.54mm_Horizontal, symbol kwp1281tool:TTL-232R-5V
- added C10: 10μF, Capacitor_SMD:C_0805_2012Metric_Pad1.18x1.45mm_HandSolder, symbol Device:C_Small
- added F1: 1206L150, Fuse:Fuse_1206_3216Metric_Pad1.42x1.75mm_HandSolder, symbol Device:Polyfuse
- added J2: USB_B, Connector_USB:USB_B_OST_USB-B1HSxx_Horizontal, symbol Connector:USB_B
- added U5: FT232RL, Package_SO:SSOP-28_5.3x10.2mm_P0.65mm, symbol Interface_USB:FT232RL
- C1, C2, C3, C6, C8, C9: footprint Capacitor_THT:C_Disc_D5.0mm_W2.5mm_P5.00mm -> Capacitor_SMD:C_0805_2012Metric_Pad1.18x1.45mm_HandSolder
Connections:
- net FTDI_GND: now also C6.1, C10.2, J2.4 (GND), U5.10 (DCD), U5.11 (CTS), U5.18 (GND), U5.21 (GND), U5.25 (AGND), U5.26 (TEST), U5.7 (GND), U5.9 (DCR)
- net FTDI_RXD: now also U5.5 (RXD)
- net FTDI_TXD: now also U5.1 (TXD)
- net FTDI_VCC: now also C6.2, C10.1, F1.2, U5.20 (VCC), U5.4 (VCCIO)
- net GND: no longer C4.1, C5.1, C6.1
- net at U3.32 (AREF): no longer C6.2
- new net: C4.1, C5.1
- new net: F1.1, J2.1 (VBUS)
- new net USB_D+: J2.3 (D+), U5.15 (USBD+)
- new net USB_D-: J2.2 (D-), U5.16 (USBD-)
- no-connect marks 29 -> 42
Other:
- note added: "C6 as close to U5 as possible"
- note added: "Differential Pair"
- note added: "Pin 9 "DCR" is "DSR" in the FT232RNL datasheet."
- moved on the sheet: C1, C2, C3, C4, C5, C7, C8, C9, D1, D2, J1, J3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

Commit message: Add pass-through circuit
Parts:
- added C11: 0.1uF, Capacitor_THT:C_Disc_D5.0mm_W2.5mm_P5.00mm, symbol Device:C_Small
- added R4: 10K, Resistor_THT:R_Axial_DIN0204_L3.6mm_D1.6mm_P7.62mm_Horizontal, symbol Device:R_Small_US
- added U6: 74LS257, Package_DIP:DIP-16_W7.62mm, symbol 74xx:74LS257
Connections:
- net GND: now also C8.2, C11.2, U6.10 (I1d), U6.11 (I0d), U6.13 (I1c), U6.14 (I0c), U6.15 (OE), U6.8 (GND); no longer C8.1
- net L9637D_RX: now also U6.6 (I1b)
- net L9637D_TX: now also U6.4 (Za); no longer R2.2, U3.17 (PD3)
- net VCC: now also C8.1, C11.1, R4.1, U6.16 (VCC); no longer C8.2
- net PASSTHRU: now reaches U3.21 (PD7)
- net PASSTHRU: now also R4.2, U6.1 (S)
- net HOST_RX renamed AVR_CTRL_RX
- net AVR_CTRL_RX: now also U6.3 (I1a)
- net HOST_TX renamed AVR_CTRL_TX
- net AVR_CTRL_TX: now also U6.5 (I0b); no longer U4.3 (INB)
- new net AVR_KLINE_TX: R2.2, U3.17 (PD3), U6.2 (I0a)
- new net ISO_RX: U4.3 (INB), U6.7 (Zb)
- no-connect marks 42 -> 43
Other:
- note added: "CBUSx and other FTDI-specific features are not used so that a different chip may be substituted if needed."
- note added: "PD6/ICP used for baud rate detection."
- note added: "Pull-up resistor puts the interface into pass-thru mode if the AVR is is not installed or is in reset."
- note added: "When PASSTHRU=1, the FT232 controls the K-line instead of the AVR."
- note removed: "L9637_RX is also connected to pin 20 (PD6/ICP) for input capture, which can be used for baud rate detection."
- note removed: "Pull-up on TX ensures no K-Line output during reset."
- moved on the sheet: C1, C10, C2, C3, C4, C5, C6, C7, C8, C9, D1, D2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
